Commit message: [models] add pepper urdf and update pr2 urdf to use ros bag

File: models/pr2.urdf (robot description, URDF)
Before this commit: robot pr2, 88 links, 87 joints
Links:
- added link head_mount_kinect2_ir_link, mass 0.1; collision sphere radius=0.0005; visual sphere radius=0.0005
- added link head_mount_kinect2_ir_optical_frame
- added link head_mount_kinect2_link, mass 0.1; collision sphere radius=0.0005; visual mesh filename=package://pr2_description/meshes/sensors/kinect2_v0/kinect2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 scale=0.001 0.001 0.001
- added link head_mount_kinect2_rgb_link, mass 0.1; collision sphere radius=0.0005; visual sphere radius=0.0005
- added link head_mount_kinect2_rgb_optical_frame
- link r_forearm_cam_optical_frame: mass 0.01 -> None
Joints:
- added joint head_mount_kinect2_ir_joint: type fixed, parent head_mount_kinect2_link, child head_mount_kinect2_ir_link, origin xyz=-0.032267 -0.0475 0.155 rpy=0.0 0.0 0.0
- added joint head_mount_kinect2_ir_optical_frame_joint: type fixed, parent head_mount_kinect2_ir_link, child head_mount_kinect2_ir_optical_frame, origin xyz=0.0 0.01 0.0 rpy=-1.57079632679 0.0 -1.57079632679
- added joint head_mount_kinect2_joint: type fixed, parent head_plate_frame, child head_mount_kinect2_link, origin xyz=-0.00632975194602 0.00630582117589 0.0891635398774 rpy=0.00490305060536 0.0261374396925 0.00113803818078
- added joint head_mount_kinect2_rgb_joint: type fixed, parent head_mount_kinect2_ir_link, child head_mount_kinect2_rgb_link, origin xyz=0.0 -0.05175 0.0 rpy=0.0 0.0 0.0
- added joint head_mount_kinect2_rgb_optical_frame_joint: type fixed, parent head_mount_kinect2_rgb_link, child head_mount_kinect2_rgb_optical_frame, origin xyz=0.0 0.0 0.0 rpy=-1.57079632679 0.0 -1.57079632679
- joint base_bellow_joint: origin xyz=-0.29 0 0.8 rpy=0 0 0 -> xyz=-0.29 0.0 0.8 rpy=0.0 0.0 0.0
- joint base_footprint_joint: origin xyz=0 0 0.051 rpy=0 0 0 -> xyz=0.0 0.0 0.051 rpy=0.0 0.0 0.0
- joint base_laser_joint: axis 0 1 0 -> 0.0 1.0 0.0; origin xyz=0.275 0.0 0.252 rpy=0 0 0 -> xyz=0.275 0.0 0.252 rpy=0.0 0.0 0.0
- joint bl_caster_l_wheel_joint: axis 0 1 0 -> 0.0 1.0 0.0; limit effort=7 velocity=15 -> effort=7.0 velocity=15.0; origin xyz=0 0.049 0 rpy=0 0 0 -> xyz=0.0 0.049 0.0 rpy=0.0 0.0 0.0
- joint bl_caster_r_wheel_joint: axis 0 1 0 -> 0.0 1.0 0.0; limit effort=7 velocity=15 -> effort=7.0 velocity=15.0; origin xyz=0 -0.049 0 rpy=0 0 0 -> xyz=0.0 -0.049 0.0 rpy=0.0 0.0 0.0
- joint bl_caster_rotation_joint: axis 0 0 1 -> 0.0 0.0 1.0; limit effort=6.5 velocity=10 -> effort=6.5 velocity=10.0; origin xyz=-0.2246 0.2246 0.0282 rpy=0 0 0 -> xyz=-0.2246 0.2246 0.0282 rpy=0.0 0.0 0.0
- joint br_caster_l_wheel_joint: axis 0 1 0 -> 0.0 1.0 0.0; limit effort=7 velocity=15 -> effort=7.0 velocity=15.0; origin xyz=0 0.049 0 rpy=0 0 0 -> xyz=0.0 0.049 0.0 rpy=0.0 0.0 0.0
- joint br_caster_r_wheel_joint: axis 0 1 0 -> 0.0 1.0 0.0; limit effort=7 velocity=15 -> effort=7.0 velocity=15.0; origin xyz=0 -0.049 0 rpy=0 0 0 -> xyz=0.0 -0.049 0.0 rpy=0.0 0.0 0.0
- joint br_caster_rotation_joint: axis 0 0 1 -> 0.0 0.0 1.0; limit effort=6.5 velocity=10 -> effort=6.5 velocity=10.0; origin xyz=-0.2246 -0.2246 0.0282 rpy=0 0 0 -> xyz=-0.2246 -0.2246 0.0282 rpy=0.0 0.0 0.0
- joint double_stereo_frame_joint: origin xyz=0.0 0.0 0.0 rpy=0 0 0 -> xyz=0.0 0.0 0.0 rpy=0.0 0.0 0.0
- joint fl_caster_l_wheel_joint: axis 0 1 0 -> 0.0 1.0 0.0; limit effort=7 velocity=15 -> effort=7.0 velocity=15.0; origin xyz=0 0.049 0 rpy=0 0 0 -> xyz=0.0 0.049 0.0 rpy=0.0 0.0 0.0
- joint fl_caster_r_wheel_joint: axis 0 1 0 -> 0.0 1.0 0.0; limit effort=7 velocity=15 -> effort=7.0 velocity=15.0; origin xyz=0 -0.049 0 rpy=0 0 0 -> xyz=0.0 -0.049 0.0 rpy=0.0 0.0 0.0
- joint fl_caster_rotation_joint: axis 0 0 1 -> 0.0 0.0 1.0; limit effort=6.5 velocity=10 -> effort=6.5 velocity=10.0; origin xyz=0.2246 0.2246 0.0282 rpy=0 0 0 -> xyz=0.2246 0.2246 0.0282 rpy=0.0 0.0 0.0
- joint fr_caster_l_wheel_joint: axis 0 1 0 -> 0.0 1.0 0.0; limit effort=7 velocity=15 -> effort=7.0 velocity=15.0; origin xyz=0 0.049 0 rpy=0 0 0 -> xyz=0.0 0.049 0.0 rpy=0.0 0.0 0.0
- joint fr_caster_r_wheel_joint: axis 0 1 0 -> 0.0 1.0 0.0; limit effort=7 velocity=15 -> effort=7.0 velocity=15.0; origin xyz=0 -0.049 0 rpy=0 0 0 -> xyz=0.0 -0.049 0.0 rpy=0.0 0.0 0.0
- joint fr_caster_rotation_joint: axis 0 0 1 -> 0.0 0.0 1.0; limit effort=6.5 velocity=10 -> effort=6.5 velocity=10.0; origin xyz=0.2246 -0.2246 0.0282 rpy=0 0 0 -> xyz=0.2246 -0.2246 0.0282 rpy=0.0 0.0 0.0
- joint head_pan_joint: axis 0 0 1 -> 0.0 0.0 1.0; limit lower=-3.007 upper=3.007 effort=2.645 velocity=6 -> lower=-3.007 upper=3.007 effort=2.645 velocity=6.0
- joint head_plate_frame_joint: origin xyz=0.0232 0 0.0645 rpy=0 0 0 -> xyz=0.0232 0.0 0.0645 rpy=0.0 0.0 0.0
- joint head_tilt_joint: axis 0 1 0 -> 0.0 1.0 0.0; limit lower=-0.471238 upper=1.39626 effort=18 velocity=5 -> lower=-0.471238 upper=1.39626 effort=18.0 velocity=5.0; origin xyz=0.068 0 0 rpy=0 0 0 -> xyz=0.068 0.0 0.0 rpy=0.0 0.0 0.0
- joint high_def_frame_joint: origin xyz=0.046457 -0.110 0.054600 rpy=0 0 0 -> xyz=0.046457 -0.11 0.0546 rpy=0.0 0.0 0.0
- joint high_def_optical_frame_joint: origin xyz=0.0            0.0         0.0 rpy=-1.57079632679 0.0 -1.57079632679 -> xyz=0.0 0.0 0.0 rpy=-1.57079632679 0.0 -1.57079632679
- joint imu_joint: axis 0 1 0 -> 0.0 1.0 0.0; origin xyz=-0.02977 -0.1497 0.164 rpy=0 3.14159265359 0 -> xyz=-0.02977 -0.1497 0.164 rpy=0.0 3.14159265359 0.0
- joint l_elbow_flex_joint: axis 0 1 0 -> 0.0 1.0 0.0; limit lower=-2.3213 upper=0.00 effort=30 velocity=3.3 -> lower=-2.3213 upper=0.0 effort=30.0 velocity=3.3; origin xyz=0.4 0 0 rpy=0 0 0 -> xyz=0.4 0.0 0.0 rpy=0.0 0.0 0.0
- joint l_forearm_cam_frame_joint: origin xyz=.135 0 .044 rpy=-1.57079632679 -0.562868683768 0 -> xyz=0.137047751739 0.00640092379884 0.0429812502876 rpy=-1.54717103906 -0.553132025225 -0.0206114263735
- joint l_forearm_cam_optical_frame_joint: origin xyz=0 0 0 rpy=-1.57079632679 0.0 -1.57079632679 -> xyz=0.0 0.0 0.0 rpy=-1.57079632679 0.0 -1.57079632679
- joint l_forearm_joint: origin xyz=0 0 0 rpy=0 0 0 -> xyz=0.0 0.0 0.0 rpy=0.0 0.0 0.0
- joint l_forearm_roll_joint: axis 1 0 0 -> 1.0 0.0 0.0; limit effort=30 velocity=3.6 -> effort=30.0 velocity=3.6; origin xyz=0 0 0 rpy=0 0 0 -> xyz=0.0 0.0 0.0 rpy=0.0 0.0 0.0
- joint l_gripper_joint: axis 0 1 0 -> 0.0 1.0 0.0; origin (none) -> xyz=0.0 0.0 0.0 rpy=0.0 0.0 0.0
- joint l_gripper_l_finger_joint: axis 0 0 1 -> 0.0 0.0 1.0; origin xyz=0.07691 0.01 0 rpy=0 0 0 -> xyz=0.07691 0.01 0.0 rpy=0.0 0.0 0.0
- joint l_gripper_l_finger_tip_joint: axis 0 0 -1 -> 0.0 0.0 -1.0; mimic joint=l_gripper_l_finger_joint multiplier=1 offset=0 -> joint=l_gripper_l_finger_joint multiplier=1.0 offset=0.0; origin xyz=0.09137 0.00495 0 rpy=0 0 0 -> xyz=0.09137 0.00495 0.0 rpy=0.0 0.0 0.0
- joint l_gripper_led_joint: origin xyz=0.0513 0.0 .0244 -> xyz=0.0513 0.0 0.0244 rpy=0.0 0.0 0.0
- joint l_gripper_motor_accelerometer_joint: origin xyz=0 0 0 rpy=0 0 0 -> xyz=0.0 0.0 0.0 rpy=0.0 0.0 0.0
- joint l_gripper_motor_screw_joint: axis 0 1 0 -> 0.0 1.0 0.0; origin xyz=0.0 0 0 rpy=0 0 0 -> xyz=0.0 0.0 0.0 rpy=0.0 0.0 0.0
- joint l_gripper_motor_slider_joint: axis 1 0 0 -> 1.0 0.0 0.0; origin xyz=0.16828 0 0 rpy=0 0 0 -> xyz=0.16828 0.0 0.0 rpy=0.0 0.0 0.0
- joint l_gripper_palm_joint: origin xyz=0 0 0 rpy=0 0 0 -> xyz=0.0 0.0 0.0 rpy=0.0 0.0 0.0
- joint l_gripper_r_finger_joint: axis 0 0 -1 -> 0.0 0.0 -1.0; mimic joint=l_gripper_l_finger_joint multiplier=1 offset=0 -> joint=l_gripper_l_finger_joint multiplier=1.0 offset=0.0; origin xyz=0.07691 -0.01 0 rpy=0 0 0 -> xyz=0.07691 -0.01 0.0 rpy=0.0 0.0 0.0
- joint l_gripper_r_finger_tip_joint: axis 0 0 1 -> 0.0 0.0 1.0; mimic joint=l_gripper_l_finger_joint multiplier=1 offset=0 -> joint=l_gripper_l_finger_joint multiplier=1.0 offset=0.0; origin xyz=0.09137 -0.00495 0 rpy=0 0 0 -> xyz=0.09137 -0.00495 0.0 rpy=0.0 0.0 0.0
- joint l_gripper_tool_joint: origin xyz=0.18 0 0 rpy=0 0 0 -> xyz=0.18 0.0 0.0 rpy=0.0 0.0 0.0
- joint l_shoulder_lift_joint: axis 0 1 0 -> 0.0 1.0 0.0; limit lower=-0.5236 upper=1.3963 effort=30 velocity=2.082 -> lower=-0.5236 upper=1.3963 effort=30.0 velocity=2.082; origin xyz=0.1 0 0 rpy=0 0 0 -> xyz=0.1 0.0 0.0 rpy=0.0 0.0 0.0
- joint l_shoulder_pan_joint: axis 0 0 1 -> 0.0 0.0 1.0; limit lower=-0.714601836603 upper=2.2853981634 effort=30 velocity=2.088 -> lower=-0.714601836603 upper=2.2853981634 effort=30.0 velocity=2.088; origin xyz=0.0 0.188 0.0 rpy=0 0 0 -> xyz=0.0 0.188 0.0 rpy=0.0 0.0 0.0
- joint l_torso_lift_side_plate_joint: origin xyz=0.0535 0.209285 0.176625 -> xyz=0.0535 0.209285 0.176625 rpy=0.0 0.0 0.0
- joint l_upper_arm_joint: origin xyz=0 0 0 rpy=0 0 0 -> xyz=0.0 0.0 0.0 rpy=0.0 0.0 0.0
- joint l_upper_arm_roll_joint: axis 1 0 0 -> 1.0 0.0 0.0; limit lower=-0.8 upper=3.9 effort=30 velocity=3.27 -> lower=-0.8 upper=3.9 effort=30.0 velocity=3.27; origin xyz=0 0 0 rpy=0 0 0 -> xyz=0.0 0.0 0.0 rpy=0.0 0.0 0.0
- joint l_wrist_flex_joint: axis 0 1 0 -> 0.0 1.0 0.0; limit lower=-2.18 upper=0.0 effort=10 velocity=3.078 -> lower=-2.18 upper=0.0 effort=10.0 velocity=3.078; origin xyz=0.321 0 0 rpy=0 0 0 -> xyz=0.321 0.0 0.0 rpy=0.0 0.0 0.0
- joint l_wrist_roll_joint: axis 1 0 0 -> 1.0 0.0 0.0; limit effort=10 velocity=3.6 -> effort=10.0 velocity=3.6; origin xyz=0 0 0 rpy=0 0 0 -> xyz=0.0 0.0 0.0 rpy=0.0 0.0 0.0
- joint laser_tilt_joint: axis 0 1 0 -> 0.0 1.0 0.0; origin xyz=0 0 0.03 rpy=0 0 0 -> xyz=0.0 0.0 0.0343702841826 rpy=0.0 0.0 -0.00956663035944
- joint laser_tilt_mount_joint: axis 0 1 0 -> 0.0 1.0 0.0; origin xyz=0.09893 0 0.227 rpy=0 0 0 -> xyz=0.09893 0.0 0.227 rpy=0.0 0.0 0.0
- joint narrow_stereo_frame_joint: origin xyz=0.045 0.06 0.0501 rpy=0.0   0.0   0.0 -> xyz=0.00823953615809 0.060373942588 0.0502666747026 rpy=-0.00156095115318 0.0390795315704 0.00927893567918
- joint narrow_stereo_l_stereo_camera_frame_joint: origin xyz=0 0 0 rpy=0 0 0 -> xyz=0.0 0.0 0.0 rpy=0.0 0.0 0.0
- joint narrow_stereo_l_stereo_camera_optical_frame_joint: origin xyz=0 0 0 rpy=-1.57079632679 0.0 -1.57079632679 -> xyz=0.0 0.0 0.0 rpy=-1.57079632679 0.0 -1.57079632679
- joint narrow_stereo_optical_frame_joint: origin xyz=0 0 0 rpy=-1.57079632679 0.0 -1.57079632679 -> xyz=0.0 0.0 0.0 rpy=-1.57079632679 0.0 -1.57079632679
- joint narrow_stereo_r_stereo_camera_optical_frame_joint: origin xyz=0 0 0 rpy=-1.57079632679 0.0 -1.57079632679 -> xyz=0.0 0.0 0.0 rpy=-1.57079632679 0.0 -1.57079632679
- joint projector_wg6802418_child_frame_joint: origin xyz=0 0 0 rpy=0 -1.57079632679 0 -> xyz=0.0 0.0 0.0 rpy=0.0 -1.57079632679 0.0
- joint projector_wg6802418_frame_joint: origin xyz=0 0.110 0.0546 rpy=0 0 0 -> xyz=0.0 0.11 0.0546 rpy=0.0 0.0 0.0
- joint r_elbow_flex_joint: axis 0 1 0 -> 0.0 1.0 0.0; limit lower=-2.3213 upper=0.00 effort=30 velocity=3.3 -> lower=-2.3213 upper=0.0 effort=30.0 velocity=3.3; origin xyz=0.4 0 0 rpy=0 0 0 -> xyz=0.4 0.0 0.0 rpy=0.0 0.0 0.0
- joint r_forearm_cam_frame_joint: origin xyz=.135 0 .044 rpy=1.57079632679 -0.562868683768 0 -> xyz=0.137914718736 -0.00440923209547 0.0442513923859 rpy=1.55096129191 -0.551037277897 0.00979745022522
- joint r_forearm_cam_optical_frame_joint: origin xyz=0 0 0 rpy=-1.57079632679 0.0 -1.57079632679 -> xyz=0.0 0.0 0.0 rpy=-1.57079632679 0.0 -1.57079632679
- joint r_forearm_joint: origin xyz=0 0 0 rpy=0 0 0 -> xyz=0.0 0.0 0.0 rpy=0.0 0.0 0.0
- joint r_forearm_roll_joint: axis 1 0 0 -> 1.0 0.0 0.0; limit effort=30 velocity=3.6 -> effort=30.0 velocity=3.6; origin xyz=0 0 0 rpy=0 0 0 -> xyz=0.0 0.0 0.0 rpy=0.0 0.0 0.0
- joint r_gripper_joint: axis 0 1 0 -> 0.0 1.0 0.0; origin (none) -> xyz=0.0 0.0 0.0 rpy=0.0 0.0 0.0
- joint r_gripper_l_finger_joint: axis 0 0 1 -> 0.0 0.0 1.0; origin xyz=0.07691 0.01 0 rpy=0 0 0 -> xyz=0.07691 0.01 0.0 rpy=0.0 0.0 0.0
- joint r_gripper_l_finger_tip_joint: axis 0 0 -1 -> 0.0 0.0 -1.0; mimic joint=r_gripper_l_finger_joint multiplier=1 offset=0 -> joint=r_gripper_l_finger_joint multiplier=1.0 offset=0.0; origin xyz=0.09137 0.00495 0 rpy=0 0 0 -> xyz=0.09137 0.00495 0.0 rpy=0.0 0.0 0.0
- joint r_gripper_led_joint: origin xyz=0.0513 0.0 .0244 -> xyz=0.0513 0.0 0.0244 rpy=0.0 0.0 0.0
- joint r_gripper_motor_accelerometer_joint: origin xyz=0 0 0 rpy=0 0 0 -> xyz=0.0 0.0 0.0 rpy=0.0 0.0 0.0
- joint r_gripper_motor_screw_joint: axis 0 1 0 -> 0.0 1.0 0.0; origin xyz=0.0 0 0 rpy=0 0 0 -> xyz=0.0 0.0 0.0 rpy=0.0 0.0 0.0
- joint r_gripper_motor_slider_joint: axis 1 0 0 -> 1.0 0.0 0.0; origin xyz=0.16828 0 0 rpy=0 0 0 -> xyz=0.16828 0.0 0.0 rpy=0.0 0.0 0.0
- joint r_gripper_palm_joint: origin xyz=0 0 0 rpy=0 0 0 -> xyz=0.0 0.0 0.0 rpy=0.0 0.0 0.0
- joint r_gripper_r_finger_joint: axis 0 0 -1 -> 0.0 0.0 -1.0; mimic joint=r_gripper_l_finger_joint multiplier=1 offset=0 -> joint=r_gripper_l_finger_joint multiplier=1.0 offset=0.0; origin xyz=0.07691 -0.01 0 rpy=0 0 0 -> xyz=0.07691 -0.01 0.0 rpy=0.0 0.0 0.0
- joint r_gripper_r_finger_tip_joint: axis 0 0 1 -> 0.0 0.0 1.0; mimic joint=r_gripper_l_finger_joint multiplier=1 offset=0 -> joint=r_gripper_l_finger_joint multiplier=1.0 offset=0.0; origin xyz=0.09137 -0.00495 0 rpy=0 0 0 -> xyz=0.09137 -0.00495 0.0 rpy=0.0 0.0 0.0
- joint r_gripper_tool_joint: origin xyz=0.18 0 0 rpy=0 0 0 -> xyz=0.18 0.0 0.0 rpy=0.0 0.0 0.0
- joint r_shoulder_lift_joint: axis 0 1 0 -> 0.0 1.0 0.0; limit lower=-0.5236 upper=1.3963 effort=30 velocity=2.082 -> lower=-0.5236 upper=1.3963 effort=30.0 velocity=2.082; origin xyz=0.1 0 0 rpy=0 0 0 -> xyz=0.1 0.0 0.0 rpy=0.0 0.0 0.0
- joint r_shoulder_pan_joint: axis 0 0 1 -> 0.0 0.0 1.0; limit lower=-2.2853981634 upper=0.714601836603 effort=30 velocity=2.088 -> lower=-2.2853981634 upper=0.714601836603 effort=30.0 velocity=2.088; origin xyz=0.0 -0.188 0.0 rpy=0 0 0 -> xyz=0.0 -0.188 0.0 rpy=0.0 0.0 0.0
- joint r_torso_lift_side_plate_joint: origin xyz=0.0535  -0.209285 0.176625 -> xyz=0.0535 -0.209285 0.176625 rpy=0.0 0.0 0.0
- joint r_upper_arm_joint: origin xyz=0 0 0 rpy=0 0 0 -> xyz=0.0 0.0 0.0 rpy=0.0 0.0 0.0
- joint r_upper_arm_roll_joint: axis 1 0 0 -> 1.0 0.0 0.0; limit lower=-3.9 upper=0.8 effort=30 velocity=3.27 -> lower=-3.9 upper=0.8 effort=30.0 velocity=3.27; origin xyz=0 0 0 rpy=0 0 0 -> xyz=0.0 0.0 0.0 rpy=0.0 0.0 0.0
- joint r_wrist_flex_joint: axis 0 1 0 -> 0.0 1.0 0.0; limit lower=-2.18 upper=0.0 effort=10 velocity=3.078 -> lower=-2.18 upper=0.0 effort=10.0 velocity=3.078; origin xyz=0.321 0 0 rpy=0 0 0 -> xyz=0.321 0.0 0.0 rpy=0.0 0.0 0.0
- joint r_wrist_roll_joint: axis 1 0 0 -> 1.0 0.0 0.0; limit effort=10 velocity=3.6 -> effort=10.0 velocity=3.6; origin xyz=0 0 0 rpy=0 0 0 -> xyz=0.0 0.0 0.0 rpy=0.0 0.0 0.0
- joint sensor_mount_frame_joint: origin xyz=0.0 0.0 0.0 rpy=0 0 0 -> xyz=0.0 0.0 0.0 rpy=0.0 0.0 0.0
- joint torso_lift_joint: axis 0 0 1 -> 0.0 0.0 1.0; limit lower=0.0 upper=0.33 effort=10000 velocity=0.013 -> lower=0.0 upper=0.33 effort=10000.0 velocity=0.013; origin xyz=-0.05 0 0.739675 rpy=0 0 0 -> xyz=-0.05 0.0 0.739675 rpy=0.0 0.0 0.0
- joint torso_lift_motor_screw_joint: axis 0 0 1 -> 0.0 0.0 1.0; origin xyz=-0.15 0.0 0.7 -> xyz=-0.15 0.0 0.7 rpy=0.0 0.0 0.0
- joint wide_stereo_frame_joint: origin xyz=0.045 0.03 0.0501 rpy=0.0   0.0   0.0 -> xyz=0.0249430650945 0.0299519756271 0.0493628985723 rpy=-0.00282534914187 0.0147453671555 0.0489744458747
- joint wide_stereo_l_stereo_camera_frame_joint: origin xyz=0 0 0 rpy=0 0 0 -> xyz=0.0 0.0 0.0 rpy=0.0 0.0 0.0
- joint wide_stereo_l_stereo_camera_optical_frame_joint: origin xyz=0 0 0 rpy=-1.57079632679 0.0 -1.57079632679 -> xyz=0.0 0.0 0.0 rpy=-1.57079632679 0.0 -1.57079632679
- joint wide_stereo_optical_frame_joint: origin xyz=0 0 0 rpy=-1.57079632679 0.0 -1.57079632679 -> xyz=0.0 0.0 0.0 rpy=-1.57079632679 0.0 -1.57079632679
- joint wide_stereo_r_stereo_camera_optical_frame_joint: origin xyz=0 0 0 rpy=-1.57079632679 0.0 -1.57079632679 -> xyz=0.0 0.0 0.0 rpy=-1.57079632679 0.0 -1.57079632679
